File: pcb/sda_evo/sda_evo.kicad_pcb (KiCad board)
At the start: 4 copper layers, 61.5 x 105.9 mm, 161 parts, among them J1 PROG, J10 SPKR, J11 AudioJack, J2 USB_C_Receptacle_USB2.0, J3 LCD_CONN, J4 INT_EXP, J5 BATT, J9 Micro_SD_Card_Det, Q1 IRLML6302, SW1 RESET, SW2 BTN_A, SW3 BTN_B, SW4 BTN_UP, SW5 BTN_DOWN, SW6 BTN_LEFT, SW7 BTN_RIGHT, SW8 BTN_PWR, U1 USBLC6, U10 STM32H743ZITx, U11 USBLC6, U12 AP22802AW5-7, U13 LM4861, U2 TLV431, U3 USBLC6, U4 AP22802AW5-7, U5 FT230XS, U6 MCP73831-2-OT, U7 PCM5102, U8 NCP1529, U9 LMR62014XMF, Y1 16Mhz, Y2 32.768

Commit message: commit before beta1
Changed lines of the file:
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@@
 		)
 		(property "Footprint" "sda-parts:SMDXT224"
-			(at 0 0 -90)
+			(at 0 0 90)
 			(layer "F.Fab")
 			(hide yes)
@@
 		)
 		(property "Datasheet" ""
-			(at 0 0 -90)
+			(at 0 0 90)
 			(layer "F.Fab")
 			(hide yes)
@@
 		)
 		(property "Description" ""
-			(at 0 0 -90)
+			(at 0 0 90)
 			(layer "F.Fab")
 			(hide yes)
@@
 		(width 0.25)
 		(layer "F.Cu")
-		(net 20)
-	)
-	(segment
-		(start 63 53.8)
-		(end 62.7 54.1)
-		(width 0.25)
-		(layer "F.Cu")

Commit message: feat: fixed b0 problems, pushed to b1
Parts:
- removed D2: 1N5819HW-7-F, Diode_SMD:D_SOD-123
- removed R38, R39, R40: 0, Resistor_SMD:R_0805_2012Metric_Pad1.20x1.40mm_HandSolder
- removed U6: MCP73831-2-OT, Package_TO_SOT_SMD:SOT-23-5_HandSoldering
- added D8: 1N5819HW-7-F, Diode_SMD:D_SOD-123, B.Cu at (82.5, 116.9)
- added D9: 1N5819HW-7-F, Diode_SMD:D_SOD-123, B.Cu at (80.1, 116.9)
- added R41: placeholder, Resistor_SMD:R_0805_2012Metric_Pad1.20x1.40mm_HandSolder, B.Cu at (80.5, 122.0)
- added R42: 10K, Resistor_SMD:R_0805_2012Metric_Pad1.20x1.40mm_HandSolder, B.Cu at (82.5, 122.0)
- added R43: 10K, Resistor_SMD:R_0805_2012Metric_Pad1.20x1.40mm_HandSolder, B.Cu at (76.0, 130.0)
- added TP10: VCAP, TestPoint:TestPoint_Pad_D1.0mm, B.Cu at (82.0, 77.7)
- added U14: STC4054, Package_TO_SOT_SMD:SOT-23-5_HandSoldering, B.Cu at (73.5, 143.4)
- C48: value 680p ? -> 680p
- D4: value 1N5819HW-7-F -> BZT52-C3V3X; footprint Diode_SMD:D_SOD-123 -> Diode_SMD:Nexperia_CFP3_SOD-123W
- D5: value 1N4148W -> S1ABF; footprint Diode_SMD:D_SOD-123 -> Diode_SMD:D_SMB
- J5: footprint Connector_PinHeader_2.54mm:PinHeader_1x02_P2.54mm_Vertical -> Connector_PinHeader_2.54mm:PinHeader_1x02_P2.54mm_Horizontal
- R13: value 19K -> 100K
- R14: value 2k -> 1k2 1%
- R31: value 20k -> 10k
- U8: footprint Package_TO_SOT_SMD:TSOT-23-5_HandSoldering -> Package_TO_SOT_SMD:SOT-23-5_HandSoldering
- moved J10 16.8 mm to (90.0, 62.0)
- moved F1 6.00 mm to (64.0, 132.8), turned to 90 degrees
- moved Q1 5.96 mm to (72.0, 134.0)
- moved R13 5.65 mm to (81.2, 134.1), turned to -90 degrees
- moved C31 3.73 mm to (75.8, 117.0), turned to -90 degrees
- moved J5 3.27 mm to (65.4, 139.7), turned to 0 degrees
- moved D4 2.57 mm to (80.6, 129.5)
- moved D5 1.85 mm to (66.2, 145.6)
- moved C41 1.82 mm to (75.2, 134.1)
- moved TP5 1.66 mm to (83.2, 134.3)
- moved R20 1.63 mm to (77.2, 134.1)
- moved C48 1.61 mm to (76.4, 123.0)
- moved R26 1.47 mm to (74.3, 123.0)
- moved R21 1.41 mm to (79.2, 134.1), turned to -90 degrees
- moved R27 1.32 mm to (72.2, 123.0)
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Connections:
- D4 pad 1: REG_EN -> BTN_PWR
- D4 pad 2: Net-(D4-A) -> GND
- F1 pad 1: Net-(J5-Pin_1) -> Net-(J5-Pin_2)
- J3 pad 38: Net-(J3-Pin_38) -> GND
- J3 pad 39: Net-(J3-Pin_39) -> +3V3
- J3 pad 40: Net-(J3-Pin_40) -> GND
- J5 pad 1: Net-(J5-Pin_1) -> GND
- J5 pad 2: GND -> Net-(J5-Pin_2)
- R12 pad 2: Net-(D4-A) -> Net-(SW8-A)
- R13 pad 1: BTN_PWR -> Net-(U9-EN)
- R20 pad 2: REG_EN -> Net-(U9-EN)
- R21 pad 1: REG_EN -> Net-(U9-EN)
- R32 pad 2: SPEAKER_PCM -> SPKR_PCM
- R36 pad 2: SPEAKER_PCM -> SPKR_PCM
- SW8 pad 1: Net-(D4-A) -> Net-(SW8-A)
- U10 pad 41: MCU_REG_EN -> MCU_3.3V_REG_EN
- U10 pad 64: unconnected-(U10-PE11-Pad64) -> MCU_5V_REG_EN
- U8 pad 1: +5V -> Net-(D8-K)
- U9 pad 4: REG_EN -> Net-(U9-EN)
- Y2 pad 1: Net-(U10-PC15) -> Net-(U10-PC14)
- Y2 pad 2: Net-(U10-PC14) -> Net-(U10-PC15)
Routing:
- net MCU_5V_REG_EN: track 0.00 -> 63.2 mm, vias 0 -> 3
- net Net-(D4-A): track 47.8 -> 0.00 mm, vias 2 -> 0
- net Net-(SW8-A): track 0.00 -> 43.0 mm, vias 0 -> 2
- net MCU_REG_EN: track 43.0 -> 0.00 mm, vias 2 -> 0
- net MCU_3.3V_REG_EN: track 0.00 -> 40.7 mm, vias 0 -> 3
- net GND: track 239.3 -> 268.0 mm, vias 67 -> 68
- net SPKR_PCM: track 8.93 -> 34.1 mm, vias 0 -> 2
- net Net-(J10-Pin_2): track 21.3 -> 42.8 mm, vias 1 -> 2
- net BTN_PWR: track 37.6 -> 57.1 mm, vias 2 -> 4
- net Net-(J10-Pin_1): track 15.0 -> 34.3 mm, vias 1 -> 2
- net Net-(D8-K): track 0.00 -> 14.4 mm
- net VBUS: track 93.7 -> 107.0 mm
- net +BATT: track 82.5 -> 95.0 mm, vias 5 -> 7
- net REG_EN: track 12.4 -> 0.00 mm
- net Net-(J3-Pin_39): track 11.3 -> 0.00 mm
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Other:
- board text added: "Beta 1 IV. 2026 Designed in Budweis by Standa"
- board text removed: "Beta 0 XII. 2025 Designed in Budweis by Standa"

Commit message: PCB updates for B1
Parts:
- added C61: 100n, Capacitor_SMD:C_0805_2012Metric_Pad1.18x1.45mm_HandSolder, F.Cu at (96.8, 72.1)
- added R38: EN_USB, Jumper:SolderJumper-2_P1.3mm_Open_TrianglePad1.0x1.5mm, F.Cu at (96.8, 76.5)
- added R39: USB_DM, Jumper:SolderJumper-2_P1.3mm_Open_TrianglePad1.0x1.5mm, F.Cu at (108.8, 130.1)
- added R40: USB_DP, Jumper:SolderJumper-2_P1.3mm_Open_TrianglePad1.0x1.5mm, F.Cu at (111.5, 130.1)
- added TP11: 3.3V, TestPoint:TestPoint_Pad_D2.5mm, F.Cu at (113.7, 69.7)
- added TP12: GND, TestPoint:TestPoint_Pad_D2.5mm, F.Cu at (113.8, 73.3)
- D3: footprint LED_THT:LED_D3.0mm_FlatTop -> sda-parts:LED_SMD_custom
- R20: value placeholder -> EN_5V; footprint Resistor_SMD:R_0805_2012Metric_Pad1.20x1.40mm_HandSolder -> Jumper:SolderJumper-2_P1.3mm_Open_TrianglePad1.0x1.5mm
- R30: value 0 -> DET0; footprint Resistor_SMD:R_0805_2012Metric_Pad1.20x1.40mm_HandSolder -> Jumper:SolderJumper-2_P1.3mm_Open_TrianglePad1.0x1.5mm
- R37: value 0 -> DET1; footprint Resistor_SMD:R_0805_2012Metric_Pad1.20x1.40mm_HandSolder -> Jumper:SolderJumper-2_P1.3mm_Open_TrianglePad1.0x1.5mm
- R41: value placeholder -> EN_3V3; footprint Resistor_SMD:R_0805_2012Metric_Pad1.20x1.40mm_HandSolder -> Jumper:SolderJumper-2_P1.3mm_Open_TrianglePad1.0x1.5mm
- TP8, TP9: moved to F.Cu
- U1, U11, U3: footprint Package_TO_SOT_SMD:TSOT-23-6_HandSoldering -> Package_TO_SOT_SMD:SOT-23-6_Handsoldering
- moved D3 4.21 mm to (84.2, 141.9)
- moved C51 1.90 mm to (62.0, 120.9), turned to 90 degrees
- moved C7 0.63 mm to (112.9, 91.1)
- moved C10 0.58 mm to (113.0, 83.9)
- moved TP10 0.50 mm to (82.0, 78.2)
- moved R37 0.50 mm to (113.0, 88.8)
- moved R30 0.36 mm to (113.0, 86.2)
- moved R21 0.35 mm to (79.6, 134.1)
- moved TP5 0.30 mm to (83.5, 134.3)
- moved U14 0.29 mm to (73.3, 143.5)
- moved R41 0.25 mm to (80.2, 122.0)
- moved R13 0.25 mm to (81.5, 134.1)
- moved F1 0.20 mm to (63.8, 132.8)
- moved U3 0.16 mm to (88.8, 142.3)
- moved R20 0.15 mm to (77.4, 134.1)
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Connections:
- C59 pad 1: Net-(C59-Pad1) -> Net-(C45-Pad1)
- C60 pad 1: Net-(C60-Pad1) -> Net-(C47-Pad1)
- J11 pad RN: Net-(C59-Pad1) -> Net-(C45-Pad1)
- J11 pad TN: Net-(C60-Pad1) -> Net-(C47-Pad1)
- R30 pad 1: GND -> +3V3
- R37 pad 1: GND -> +3V3
- U10 pad 103: unconnected-(U10-PA11-Pad103) -> MCU_USB_DM
- U10 pad 104: unconnected-(U10-PA12-Pad104) -> MCU_USB_DP
- U10 pad 95: unconnected-(U10-VDD33_USB-Pad95) -> Net-(U10-VDD33_USB)
Routing:
- net MCU_USB_DM: track 0.00 -> 66.3 mm, vias 0 -> 1
- net MCU_USB_DP: track 0.00 -> 58.4 mm, vias 0 -> 1
- net Net-(C45-Pad1): track 25.9 -> 35.4 mm, vias 2 -> 3
- net +3V3: track 491.7 -> 500.5 mm
- net Net-(C59-Pad1): track 6.86 -> 0.00 mm, vias 1 -> 0
- net Net-(C47-Pad1): track 18.3 -> 24.3 mm, vias 2 -> 3
- net GND: track 268.0 -> 262.9 mm
- net Net-(C60-Pad1): track 4.68 -> 0.00 mm, vias 1 -> 0
- net Net-(D3-K): track 5.34 -> 8.84 mm
- net Net-(U10-VDD33_USB): track 0.00 -> 3.41 mm, vias 0 -> 1
- net Net-(R39-Pad2): track 35.8 -> 38.9 mm
- net BTN_UP: track 80.3 -> 82.9 mm
- net Net-(R40-Pad2): track 36.0 -> 38.5 mm
- net +5V: track 116.7 -> 118.7 mm
- net Net-(U9-FB): track 10.5 -> 8.96 mm
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Other:
- outline, holes or cut-outs redrawn
- board text added: "Beta 1 V. 2026 Designed in Budweis by Standa"
- board text removed: "Beta 1 IV. 2026 Designed in Budweis by Standa"
