File: pcb/sda_evo/sda_evo.kicad_sch (KiCad schematic)
At the start: 136 parts, among them J1 PROG, J10 SPKR, J11 AudioJack, J2 USB_C_Receptacle_USB2.0, J3 Conn_01x40, J4 INT_EXP, J5 BATT, J9 Micro_SD_Card_Det, Q1 IRLML6302, SW1 RESET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

Commit message: Adaded part mockups. PCB is nearly finished.
Parts:
- added C52: 100n, Capacitor_SMD:C_0805_2012Metric_Pad1.18x1.45mm_HandSolder, symbol Device:C
- added C53: 4.7u, Capacitor_SMD:C_0805_2012Metric_Pad1.18x1.45mm_HandSolder, symbol Device:C
- C22, C23: value ?? -> 12,5p
- C3, C4: value ?? -> 12p
- J2: footprint Connector_USB:USB_C_Receptacle_XKB_U262-16XN-4BVC11 -> sda-parts:USB_C
- SW1: footprint Button_Switch_SMD:SW_SPST_B3S-1000 -> Button_Switch_SMD:SW_SPST_PTS645
- TP2: value TP_VUSB -> VUSB
Connections:
- net +3V3: now also C52.1, C53.1
- net BTN_A: now also U10.27 (PC1); no longer U10.26 (PC0)
- net BTN_B: now also U10.26 (PC0); no longer U10.27 (PC1)
- net GND: now also C52.2, C53.2
- net LCD_CS: now also U10.4 (PE5)
- net LCD_RD: now also U10.59 (PE8); no longer U10.128 (PG13)
- net LCD_RS: now also U10.63 (PE10); no longer U10.132 (PG15)
- net LCD_RST: now also U10.58 (PE7); no longer U10.127 (PG12)
- net LCD_WR: now also U10.60 (PE9); no longer U10.129 (PG14)
- net TS_P1: now also U10.56 (PG0); no longer U10.139 (PB8)
- net TS_P2: now also U10.57 (PG1); no longer U10.140 (PB9)
- no-connect marks 50 -> 45

Commit message: PCB: footprints adjusted
Parts:
- C22, C23: value 12,5p -> 15p
- C3, C4: value 12p -> 15p
Other:
- moved on the sheet: C1, C10, C11, C12, C13, C14, C15, C16, C17, C2, C21, C5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

Commit message: did some stuff
Parts:
- added C54, C56: 100n, Capacitor_SMD:C_0805_2012Metric_Pad1.18x1.45mm_HandSolder, symbol Device:C
- added C55: 1u, Capacitor_SMD:C_0805_2012Metric_Pad1.18x1.45mm_HandSolder, symbol Device:C
- added C57: 2.2u, Capacitor_SMD:C_0805_2012Metric_Pad1.18x1.45mm_HandSolder, symbol Device:C
- added C58, C59, C60: 390n, Capacitor_SMD:C_0805_2012Metric_Pad1.18x1.45mm_HandSolder, symbol Device:C
- added R31, R32, R35, R36: 20k, Resistor_SMD:R_0805_2012Metric_Pad1.20x1.40mm_HandSolder, symbol Device:R
- added R33: 10k, Resistor_SMD:R_0805_2012Metric_Pad1.20x1.40mm_HandSolder, symbol Device:R
- added R34: R_Photo, LED_THT:LED_D5.0mm, symbol Device:R_Photo
- added TP6: AUX_SW, TestPoint:TestPoint_Pad_D2.5mm, symbol Connector:TestPoint
- added TP7: AUX_GND, TestPoint:TestPoint_Pad_D2.5mm, symbol Connector:TestPoint
- added TP8: PD3, TestPoint:TestPoint_Pad_D2.5mm, symbol Connector:TestPoint
- added TP9: PD4, TestPoint:TestPoint_Pad_D2.5mm, symbol Connector:TestPoint
- added U12: AP22802AW5-7, Package_TO_SOT_SMD:SOT-23-5_HandSoldering, symbol Power_Management:AP22804AW5
- added U13: ~, Package_SO:HSOP-8-1EP_3.9x4.9mm_P1.27mm_EP2.41x3.1mm, symbol sda-custom-parts:LM4861
- C48: value ?? -> 660p ?
- SW1: footprint Button_Switch_SMD:SW_SPST_PTS645 -> sda-parts:SW_SPST_RESET
- SW8: footprint Button_Switch_SMD:SW_Push_1P1T_NO_CK_KMR2 -> sda-parts:SW_Push_1P1T_NO_CK_KMR2_PWR
Connections:
- net +3V3: now also R33.2, U12.5 (IN)
- net +5V: now also C54.1, U13.6 (VDD)
- net BTN_A: now also U10.45 (PC5); no longer U10.27 (PC1)
- net BTN_RIGHT: now also U10.27 (PC1); no longer U10.45 (PC5)
- net GND: now also C56.2, C57.2, R34.2, TP7.1, U12.2 (GND)
- net GNDA: now also C54.2, C55.2, U13.7 (GND); no longer J10.2 (Pin_2)
- net AUX_SWITCH: now reaches U10.1 (PE2)
- net AUX_SWITCH: now also U12.4 (EN)
- net at U10.114 (PD0): now also TP8.1
- net at U10.115 (PD1): now also TP9.1
- net AMB_SENS: now reaches U10.40 (PA4)
- net AMB_SENS: now also R33.1, R34.1
- net IEXP2_P10 renamed SPKR_SHDN
- net SPKR_SHDN: now also U13.1 (SHDN)
- net IEXP2_P9 renamed BEEPER
- net BEEPER: now also C58.1
- new net: C55.1, U13.2 (BYPASS), U13.3 (+IN)
- new net: J10.2 (Pin_2), R31.2, U13.5 (Vo1)
- new net: J10.1 (Pin_1), U13.8 (Vo2)
- new net: C59.1, J11.RN
- new net: C59.2, R32.1
- new net: C60.1, J11.TN
- new net: C60.2, R36.1
- new net: C58.2, R35.1
- new net: C56.1, C57.1, TP6.1, U12.1 (OUT)
- new net SPEAKER_PCM: R32.2, R36.2
- new net SPKR_PCM: R31.1, R35.2, U13.4 (-IN)
- no-connect marks 45 -> 42
Other:
- note added: "TIM15_CH2"
- note added: "TIM4_CH3"
- note added: "USART4"
- note added: "USART8"
- note added: "Vref"
- moved on the sheet: C19, C22, C23, C3, C4, C6, C8, D7, H1, H2, H3, H4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

Commit message: repo cleanup, board twaked
Parts:
- removed R30: 0, Resistor_SMD:R_0805_2012Metric_Pad1.20x1.40mm_HandSolder, symbol Device:R
- C48: value 660p ? -> 680p ?
- J3: value Conn_01x40 -> LCD_CONN
- U13: value ~ -> LM4861
- renumbered IEXP1 to EXP1
Connections:
- net GNDA is gone; now on net GND: C36.2, C42.2, C44.2, C45.2, C47.2, C54.2, C55.2, J11.S, U13.7 (GND), U7.3 (CPGND), U7.9 (AGND)
Other:
- note added: "40k2 will give about 4.95V output voltage and 93uA divider current orig C=660, but value was out of stock.."
- note removed: "40k2 will give about 4.95V output voltage and 93uA divider current"

Commit message: datasheets cleanup, pcb finalized
Parts:
- added R30, R37, R38, R39, R40: 0, Resistor_SMD:R_0805_2012Metric_Pad1.20x1.40mm_HandSolder, symbol Device:R
Connections:
- net +3V3: now also R40.1; no longer J3.39 (Pin_39)
- net GND: now also R30.1, R37.1, R38.1, R39.1; no longer J3.38 (Pin_38), J3.40 (Pin_40)
- net at U10.124 (PG9): now also R30.2
- net at U10.125 (PG10): now also R37.2
- new net: J3.38 (Pin_38), R39.2
- new net: J3.39 (Pin_39), R40.2
- new net: J3.40 (Pin_40), R38.2
- no-connect marks 42 -> 44
Other:
- note added: "Rev Detect: 0: unpopulated"
- note added: "note: 330pF"

Commit message: commit before beta1
Parts:
- C48: value 680p ? -> 680p
Connections:
- net SPEAKER_PCM is gone; now on net SPKR_PCM: R32.2, R36.2
Other:
- note added: "10K - 20K was too loud..."
- note added: "Change to STC4054GR for 800mA charge, verify charge circuit"
- note added: "If VD goes under 3,3V, D4 will pass 3,3V on VD, then the 3,3V rail falls... (after modif pwrbtn from vcc)"
- note added: "REG_EN does not work as expected, VD just flows to +5V. Better shutdown circuit is needed."
- note added: "SW shutdown can be implemeted here, get EN to low and also shutdown the 5V"
- note added: "This is a problem, on 2.7V VD, BTN_PWR is 1,7V and the button stops working"
- note added: "USB_OTG"
- note added: "replace with mmbd4448-7-f or similar"

Commit message: feat: fixed b0 problems, pushed to b1
Parts:
- removed D2, D4: 1N5819HW-7-F, Diode_SMD:D_SOD-123, symbol Device:D_Schottky
- removed R38, R39, R40: 0, Resistor_SMD:R_0805_2012Metric_Pad1.20x1.40mm_HandSolder, symbol Device:R
- removed U6: MCP73831-2-OT, Package_TO_SOT_SMD:SOT-23-5_HandSoldering, symbol Battery_Management:MCP73831-2-OT
- added D4: BZT52-C3V3X, Diode_SMD:Nexperia_CFP3_SOD-123W, symbol Device:D_Zener
- added D8, D9: 1N5819HW-7-F, Diode_SMD:D_SOD-123, symbol Device:D_Schottky
- added R41: placeholder, Resistor_SMD:R_0805_2012Metric_Pad1.20x1.40mm_HandSolder, symbol Device:R
- added R42, R43: 10K, Resistor_SMD:R_0805_2012Metric_Pad1.20x1.40mm_HandSolder, symbol Device:R
- added TP10: VCAP, TestPoint:TestPoint_Pad_D1.0mm, symbol Connector:TestPoint
- added U14: STC4054, Package_TO_SOT_SMD:SOT-23-5_HandSoldering, symbol sda-custom-parts:STC4054
- D5: value 1N4148W -> S1ABF; footprint Diode_SMD:D_SOD-123 -> Diode_SMD:D_SMB
- J5: footprint Connector_PinHeader_2.54mm:PinHeader_1x02_P2.54mm_Vertical -> Connector_PinHeader_2.54mm:PinHeader_1x02_P2.54mm_Horizontal
- R13: value 19K -> 100K
- R14: value 2k -> 1k2 1%
- R31: value 20k -> 10k
- U8: footprint Package_TO_SOT_SMD:TSOT-23-5_HandSoldering -> Package_TO_SOT_SMD:SOT-23-5_HandSoldering
- Y1: symbol Device:Crystal -> Device:Crystal_GND3
Connections:
- net +3V3: now also J3.39 (Pin_39)
- net +5V: now also R41.1; no longer U8.1 (EN)
- net +BATT: now also U14.3 (BAT)
- net BTN_PWR: now also D4.1 (K), D9.2 (A); no longer R13.1
- net GND: now also J3.38 (Pin_38), J3.40 (Pin_40), J5.1 (Pin_1), Y1.3, D4.2 (A), R42.2, U14.2 (GND); no longer J5.2 (Pin_2)
- net VBUS: now also U14.4 (VCC)
- net MCU_5V_REG_EN: now reaches U10.64 (PE11)
- net MCU_5V_REG_EN: now also R43.1
- net at C6.1, U10.71 (VCAP1): now also TP10.1
- net at C22.2, U10.8 (PC14): now also Y2.1; no longer Y2.2
- net at C23.2, U10.9 (PC15): now also Y2.2; no longer Y2.1
- net at F1.1: now also J5.2 (Pin_2); no longer J5.1 (Pin_1)
- net at R10.2, R9.1: now also U14.1 (CHRG)
- net at R14.2: now also U14.5 (PROG)
- net MCU_REG_EN renamed MCU_3.3V_REG_EN
- net MCU_3.3V_REG_EN: now also D8.2 (A)
- net REG_EN: no longer names the net of R20.2, R21.1, U9.4 (EN)
- net REG_EN: now also R13.1, R43.2
- new net: D8.1 (K), D9.1 (K), R41.2, R42.1, U8.1 (EN)
- no-connect marks 44 -> 43
Other:
- note added: "2026-04-19"
- note added: "3.3 - 2.7V"
- note added: "Beta 1"
- note removed: "10K - 20K was too loud..."
- note removed: "Change to STC4054GR for 800mA charge, verify charge circuit"
- note removed: "If VD goes under 3,3V, D4 will pass 3,3V on VD, then the 3,3V rail falls... (after modif pwrbtn from vcc)"
- note removed: "REG_EN does not work as expected, VD just flows to +5V. Better shutdown circuit is needed."
- note removed: "SW shutdown can be implemeted here, get EN to low and also shutdown the 5V"
- note removed: "This is a problem, on 2.7V VD, BTN_PWR is 1,7V and the button stops working"
- note removed: "replace with mmbd4448-7-f or similar"
- moved on the sheet: C19, C20, C22, C23, C27, C3, C31, C33, C39, C4, C41, C46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

Commit message: PCB updates for B1
Parts:
- added C61: 100n, Capacitor_SMD:C_0805_2012Metric_Pad1.18x1.45mm_HandSolder, symbol Device:C
- added R38: EN_USB, Jumper:SolderJumper-2_P1.3mm_Open_TrianglePad1.0x1.5mm, symbol Device:R
- added R39: USB_DM, Jumper:SolderJumper-2_P1.3mm_Open_TrianglePad1.0x1.5mm, symbol Device:R
- added R40: USB_DP, Jumper:SolderJumper-2_P1.3mm_Open_TrianglePad1.0x1.5mm, symbol Device:R
- added TP11: 3.3V, TestPoint:TestPoint_Pad_D2.5mm, symbol Connector:TestPoint
- added TP12: GND, TestPoint:TestPoint_Pad_D2.5mm, symbol Connector:TestPoint
- D3: footprint LED_THT:LED_D3.0mm_FlatTop -> sda-parts:LED_SMD_custom
- R20: value placeholder -> EN_5V; footprint Resistor_SMD:R_0805_2012Metric_Pad1.20x1.40mm_HandSolder -> Jumper:SolderJumper-2_P1.3mm_Open_TrianglePad1.0x1.5mm
- R30: value 0 -> DET0; footprint Resistor_SMD:R_0805_2012Metric_Pad1.20x1.40mm_HandSolder -> Jumper:SolderJumper-2_P1.3mm_Open_TrianglePad1.0x1.5mm
- R37: value 0 -> DET1; footprint Resistor_SMD:R_0805_2012Metric_Pad1.20x1.40mm_HandSolder -> Jumper:SolderJumper-2_P1.3mm_Open_TrianglePad1.0x1.5mm
- R41: value placeholder -> EN_3V3; footprint Resistor_SMD:R_0805_2012Metric_Pad1.20x1.40mm_HandSolder -> Jumper:SolderJumper-2_P1.3mm_Open_TrianglePad1.0x1.5mm
- U1, U11, U3: footprint Package_TO_SOT_SMD:TSOT-23-6_HandSoldering -> Package_TO_SOT_SMD:SOT-23-6_Handsoldering
Connections:
- net +3V3: now also R30.1, R37.1, C61.1, R38.1, TP11.1
- net GND: now also C61.2, TP12.1; no longer R30.1, R37.1
- net at C47.1, J11.T, R24.2: now also C60.1, J11.TN
- net at C59.1, J11.RN: now also C45.1, J11.R, R25.2
- net MCU_USB_DM: now reaches U10.103 (PA11)
- net MCU_USB_DM: now also R39.1
- net MCU_USB_DP: now reaches U10.104 (PA12)
- net MCU_USB_DP: now also R40.1
- net at U10.95 (VDD33_USB): now also R38.2
- net at R8.1, U3.4 (I/02): now also R40.2
- net at R7.1, U3.6 (I/01): now also R39.2
- no-connect marks 43 -> 40
Other:
- moved on the sheet: R30, R7, R8
