File: pcb/sda_evo/sda_evo.kicad_sch (KiCad schematic)
At the start: 169 parts, among them J1 PROG, J10 SPKR, J11 AudioJack, J2 USB_C_Receptacle_USB2.0, J3 LCD_CONN, J4 INT_EXP, J5 BATT, J9 Micro_SD_Card_Det, Q1 IRLML6302, SW1 RESET, SW2 BTN_A, SW3 BTN_B, SW4 BTN_UP, SW5 BTN_DOWN, SW6 BTN_LEFT, SW7 BTN_RIGHT, SW8 BTN_PWR, U1 USBLC6, U10 STM32H743ZITx, U11 USBLC6, U12 AP22802AW5-7, U13 LM4861, U14 STC4054, U2 TLV431, U3 USBLC6, U4 AP22802AW5-7, U5 FT230XS, U7 PCM5102, U8 NCP1529, U9 LMR62014XMF, Y1 16Mhz, Y2 32.768

Commit message: feat: beta1
Parts:
- R42, R43: value 10K -> 10k
Changed lines of the file:
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@@
 		(fields_autoplaced yes)
 		(property "Reference" "R1"
-			(at 32.385 45.7199 0)
+			(at 31.75 45.7199 0)
 			(effects
 				(font
@@
 		)
 		(property "Value" "10k"
-			(at 32.385 48.2599 0)
+			(at 31.75 48.2599 0)
 			(effects
 				(font
@@
 			)
 		)
-		(property "Value" "10K"
+		(property "Value" "10k"
 			(at 492.76 327.66 0)
 			(effects
@@
 			)
 		)
-		(property "Value" "10K"
+		(property "Value" "10k"
 			(at 483.87 241.2999 0)
 			(effects
